File: connector-main-computer/connector-main-computer.kicad_pcb (KiCad board)
At the start: 2 copper layers, 97.3 x 100.3 mm, 62 parts, among them J1 DVI-I_Dual_Link, J10 Conn_01x04_MountingPin, J11 Conn_01x04_MountingPin, J12 Conn_01x02_MountingPin, J13 Conn_01x04_MountingPin, J2 Conn_01x03_MountingPin, J3 Conn_01x03_MountingPin, J4 Conn_01x03_MountingPin, J5 Conn_01x03_MountingPin, J6 Conn_01x03_MountingPin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

Commit message: Add labels on port
Other:
- board text added: "Battery Sense"
- board text added: "Big Fucking Connector"
- board text added: "I2C"
- board text added: "Preasure 1"
- board text added: "Preasure 2"
- board text added: "SMAAART Transmit"
- board text added: "Safety Switch"
- board text added: "Safety Switch Sense"
- board text added: "Servo PWM"
- board text added: "Starter Sense"
- board text added: "Strain Gauge"
- board text added: "UART"
Changed lines of the file:
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@@
 		(layer "Edge.Cuts")
+	)
+	(gr_text "Strain\nGauge"
+		(at 133 98.6 90)
+		(layer "B.SilkS")
+		(effects
+			(font
+				(size 1.5 1.5)
+				(thickness 0.3)
+				(bold yes)
+			)
+			(justify left bottom mirror)
+		)
+	)
+	(gr_text "Safety\nSwitch"
+		(at 41 84.2 270)
+		(layer "B.SilkS")
+		(effects
+			(font
+				(size 1.5 1.5)
+				(thickness 0.3)
+				(bold yes)
+			)
+			(justify left bottom mirror)
+		)
+	)
+	(gr_text "Preasure 1"
+		(at 131.8 65.3 90)
+		(layer "B.SilkS")
+		(effects
+			(font
+				(size 1.5 1.5)
+				(thickness 0.3)
+				(bold yes)
+			)
+			(justify left bottom mirror)
+		)
+	)
+	(gr_text "SMAAART\nTransmit"
+		(at 41.4 117 270)
+		(layer "B.SilkS")
+		(effects
+			(font
+				(size 1.5 1.5)
+				(thickness 0.3)
+				(bold yes)
+			)
+			(justify left bottom mirror)
+		)
+	)
+	(gr_text "Preasure 2"
+		(at 131.8 80.9 90)
+		(layer "B.SilkS")
+		(effects
+			(font
+				(size 1.5 1.5)
+				(thickness 0.3)
+				(bold yes)
+			)
+			(justify left bottom mirror)
+		)
+	)
+	(gr_text "I2C"
+		(at 110.2 143.9 0)
+		(layer "B.SilkS")
+		(effects
+			(font
+				(size 1.5 1.5)
+				(thickness 0.3)
+				(bold yes)
+			)
+			(justify left bottom mirror)
+		)
+	)
+	(gr_text "Starter\nSense"
+		(at 133.5 127.2 90)
+		(layer "B.SilkS")
+		(effects
+			(font
+				(size 1.5 1.5)
+				(thickness 0.3)
+				(bold yes)
+			)
+			(justify left bottom mirror)
+		)
+	)
+	(gr_text "Big Fucking \nConnector"
+		(at 78.4 58.6 180)
+		(layer "B.SilkS")
+		(effects
+			(font
+				(size 1.5 1.5)
+				(thickness 0.3)
+				(bold yes)
+			)
+			(justify left bottom mirror)
+		)
+	)
+	(gr_text "Servo\nPWM"
+		(at 41.7 133 270)
+		(layer "B.SilkS")
+		(effects
+			(font
+				(size 1.5 1.5)
+				(thickness 0.3)
+				(bold yes)
+			)
+			(justify left bottom mirror)
+		)
+	)
+	(gr_text "Safety\nSwitch\nSense"
+		(at 40.5 98.5 270)
+		(layer "B.SilkS")
+		(effects
+			(font
+				(size 1.5 1.5)
+				(thickness 0.3)
+				(bold yes)
+			)
+			(justify left bottom mirror)
+		)
+	)
+	(gr_text "UART"
+		(at 75.9 143.6 0)
+		(layer "B.SilkS")
+		(effects
+			(font
+				(size 1.5 1.5)
+				(thickness 0.3)
+				(bold yes)
+			)
+			(justify left bottom mirror)
+		)
+	)
+	(gr_text "I2C"
+		(at 95.1 143.9 0)
+		(layer "B.SilkS")
+		(effects
+			(font
+				(size 1.5 1.5)
+				(thickness 0.3)
+				(bold yes)
+			)
+			(justify left bottom mirror)
+		)
+	)
+	(gr_text "Battery\nSense"
+		(at 132.9 113.1 90)
+		(layer "B.SilkS")
+		(effects
+			(font
+				(size 1.5 1.5)
+				(thickness 0.3)
+				(bold yes)
+			)
+			(justify left bottom mirror)
+		)
 	)
 	(gr_text_box "${PROJECTNAME} ${CURRENT_DATE}"
