File: connector-test-stand/connector-test-stand.kicad_sch (KiCad schematic)
At the start: 85 parts, among them J1 Conn_01x02, J10 Conn_01x04_MountingPin, J11 DE9_Socket_MountingHoles, J12 DVI-I_Dual_Link, J2 Conn_01x02, J3 Conn_01x02, J4 Conn_01x05, J5 Conn_01x04_MountingPin, J6 Conn_01x02, J7 Conn_01x03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

Commit message: updates
Parts:
- R1, R2, R3, R4, R5, R6: value R -> 0
- U10: value SN65HVD11HD -> SN65HVD485E
Changed lines of the file:
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@@
 		(fields_autoplaced yes)
 		(property "Reference" "R2"
-			(at 38.608 365.8178 0)
+			(at 39.37 365.7599 0)
 			(effects
 				(font
@@
 			)
 		)
-		(property "Value" "R"
-			(at 38.608 368.2421 0)
+		(property "Value" "0"
+			(at 39.37 368.2999 0)
 			(effects
 				(font
@@
 		(fields_autoplaced yes)
 		(property "Reference" "U10"
-			(at 353.9333 276.5255 0)
+			(at 353.9333 275.59 0)
 			(effects
 				(font
@@
 			)
 		)
-		(property "Value" "SN65HVD11HD"
-			(at 353.9333 278.9498 0)
+		(property "Value" "SN65HVD485E"
+			(at 353.9333 278.13 0)
 			(effects
 				(font
@@
 		(fields_autoplaced yes)
 		(property "Reference" "R6"
-			(at 51.308 365.8178 0)
+			(at 52.07 365.7599 0)
 			(effects
 				(font
@@
 			)
 		)
-		(property "Value" "R"
-			(at 51.308 368.2421 0)
+		(property "Value" "0"
+			(at 52.07 368.2999 0)
 			(effects
 				(font
@@
 		(fields_autoplaced yes)
 		(property "Reference" "R1"
-			(at 38.608 345.4978 0)
+			(at 39.37 345.4399 0)
 			(effects
 				(font
@@
 			)
 		)
-		(property "Value" "R"
-			(at 38.608 347.9221 0)
+		(property "Value" "0"
+			(at 39.37 347.9799 0)
 			(effects
 				(font
@@
 		(fields_autoplaced yes)
 		(property "Reference" "R4"
-			(at 44.958 365.8178 0)
+			(at 45.72 365.7599 0)
 			(effects
 				(font
@@
 			)
 		)
-		(property "Value" "R"
-			(at 44.958 368.2421 0)
+		(property "Value" "0"
+			(at 45.72 368.2999 0)
 			(effects
 				(font
@@
 		(fields_autoplaced yes)
 		(property "Reference" "R5"
-			(at 51.308 345.4978 0)
+			(at 52.07 345.4399 0)
 			(effects
 				(font
@@
 			)
 		)
-		(property "Value" "R"
-			(at 51.308 347.9221 0)
+		(property "Value" "0"
+			(at 52.07 347.9799 0)
 			(effects
 				(font
@@
 		(fields_autoplaced yes)
 		(property "Reference" "R3"
-			(at 44.958 345.4978 0)
+			(at 45.72 345.4399 0)
 			(effects
 				(font
@@
 			)
 		)
-		(property "Value" "R"
-			(at 44.958 347.9221 0)
+		(property "Value" "0"
+			(at 45.72 347.9799 0)
 			(effects
 				(font
@@
 		(fields_autoplaced yes)
 		(property "Reference" "C11"
-			(at 236.601 95.3078 0)
+			(at 237.49 95.2499 0)
 			(effects
 				(font
