File: blackbox/blackbox.kicad_sch (KiCad schematic)
At the start: 55 parts, among them J1 Micro_SD_Card_Det2, J2 Conn_01x04_MountingPin, J3 Conn_02x05_Odd_Even, J4 Barrel_Jack_Switch, SW1 SW_SPST, SW2 SW_SPST, U1 STM32C011F4Px, U11 MAX811TEUS-T, U2 HCPL-063A, U3 HCPL-063A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

Commit message: blackbox update
Parts:
- added R13, R14: 10k, Resistor_SMD:R_0805_2012Metric, symbol Device:R
- R3, R4: value R -> 220R
- Y1: value Crystal_GND24 -> 16Mhz
Connections:
- net +3.3V: now also R13.2, R14.1
- net GND: now also U3.3 (C2); no longer U3.4 (A2)
- net GND1: now also U2.3 (C2); no longer U2.4 (A2)
- net at R6.2: now also U2.4 (A2); no longer U2.3 (C2)
- net at R4.1: now also U3.4 (A2); no longer U3.3 (C2)
- net at J1.1 (DAT2): now also R13.1
- net at J1.8 (DAT1): now also R14.2
- no-connect marks 8 -> 6
Other:
- moved on the sheet: R3, R4, R6, SW1

Commit message: Blackbox update
Parts:
- removed BT1: 1051, keys1051:BAT_1051, symbol keys1051:1051
- added J5: Conn_01x02_MountingPin, Connector_JST:JST_PH_S2B-PH-SM4-TB_1x02-1MP_P2.00mm_Horizontal, symbol Connector_Generic_MountingPin:Conn_01x02_MountingPin
- added SW3: SW_DPDT_x2, Button_Switch_SMD:SW_DPDT_CK_JS202011JCQN, symbol Switch:SW_DPDT_x2
Connections:
- net GND: now also J5.2 (Pin_2), J5.MP (MountPin)
- net VDD: now also SW3.1 (A)
- new net: J5.1 (Pin_1), SW3.2 (B)
- no-connect marks 6 -> 7
Other:
- moved on the sheet: C13, R10, R11

Commit message: Add NOT gate to fix uart, rework silkscreen
Parts:
- added C18: 100nF, Capacitor_SMD:C_0805_2012Metric, symbol Device:C
- added U7: 74AHCT1G04, Package_TO_SOT_SMD:SOT-23-5, symbol 74xGxx:74AHCT1G04
Connections:
- net +3.3V: now also C18.1, U7.5 (VCC)
- net ESP_TX: now also U7.4; no longer U2.7 (VO1)
- net GND: now also C18.2, U7.3 (GND)
- new net: U2.7 (VO1), U7.2

Commit message: Add more capacitors as SD cards are hungry when hotswapped
Parts:
- added C19, C20: 47uF, Capacitor_SMD:C_1206_3216Metric, symbol Device:C
- added R15: 10K, Resistor_SMD:R_0805_2012Metric, symbol Device:R
Connections:
- net +3.3V: now also C19.1, C20.1, R15.1
- net GND: now also C19.2, C20.2
- net at U2.7 (VO1), U7.2: now also R15.2
